Commit message: level3

File: urdf/fp3_2.urdf (robot description, URDF)
Before this commit: robot fp3, 14 links, 13 joints
Links:
- removed link base
- removed link fp3_hand
- removed link fp3_hand_tcp
- removed link fp3_leftfinger
- removed link fp3_link0
- removed link fp3_link1
- removed link fp3_link2
- removed link fp3_link3
- removed link fp3_link4
- removed link fp3_link5
- removed link fp3_link6
- removed link fp3_link7
- removed link fp3_link8
- removed link fp3_rightfinger
- added link fp3_2_base
- added link fp3_2_hand, mass 0.6544; collision mesh filename=package://robot_descriptions/meshes/robot_ee/franka_hand_bl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; visual mesh filename=package://robot_descriptions/meshes/robot_ee/franka_hand_bl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
- added link fp3_2_hand_tcp
- added link fp3_2_leftfinger, mass 0.0291; collision box size=17.5e-3 15.2e-3 18.5e-3; collision box size=17.5e-3 7e-3 23.5e-3
- added link fp3_2_link0, mass 2.3966; collision mesh filename=package://robot_descriptions/meshes/robot_arms/fp3/collisio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; visual mesh filename=package://robot_descriptions/meshes/robot_arms/fp3/visual/l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
- added link fp3_2_link1, mass 2.9274653454; collision mesh filename=package://robot_descriptions/meshes/robot_arms/fp3/collisio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; visual mesh filename=package://robot_descriptions/meshes/robot_arms/fp3/visual/l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
- added link fp3_2_link2, mass 2.9355370338; collision mesh filename=package://robot_descriptions/meshes/robot_arms/fp3/collisio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; visual mesh filename=package://robot_descriptions/meshes/robot_arms/fp3/visual/l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
- added link fp3_2_link3, mass 2.2449013699; collision mesh filename=package://robot_descriptions/meshes/robot_arms/fp3/collisio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; visual mesh filename=package://robot_descriptions/meshes/robot_arms/fp3/visual/l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
- added link fp3_2_link4, mass 2.6155955791; collision mesh filename=package://robot_descriptions/meshes/robot_arms/fp3/collisio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; visual mesh filename=package://robot_descriptions/meshes/robot_arms/fp3/visual/l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
- added link fp3_2_link5, mass 2.3271207594; collision mesh filename=package://robot_descriptions/meshes/robot_arms/fp3/collisio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; visual mesh filename=package://robot_descriptions/meshes/robot_arms/fp3/visual/l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
- added link fp3_2_link6, mass 1.8170376524; collision mesh filename=package://robot_descriptions/meshes/robot_arms/fp3/collisio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; visual mesh filename=package://robot_descriptions/meshes/robot_arms/fp3/visual/l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
- added link fp3_2_link7, mass 0.6271432862; collision mesh filename=package://robot_descriptions/meshes/robot_arms/fp3/collisio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; visual mesh filename=package://robot_descriptions/meshes/robot_arms/fp3/visual/l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
- added link fp3_2_link8
- added link fp3_2_rightfinger, mass 0.0291; collision box size=17.5e-3 15.2e-3 18.5e-3; collision box size=17.5e-3 7e-3 23.5e-3
Joints:
- removed joint fp3_base_joint
- removed joint fp3_finger_joint1
- removed joint fp3_finger_joint2
- removed joint fp3_hand_joint
- removed joint fp3_hand_tcp_joint
- removed joint fp3_joint1
- removed joint fp3_joint2
- removed joint fp3_joint3
- removed joint fp3_joint4
- removed joint fp3_joint5
- removed joint fp3_joint6
- removed joint fp3_joint7
- removed joint fp3_joint8
- added joint fp3_2_base_joint: type fixed, parent fp3_2_base, child fp3_2_link0, origin xyz=0 0 0 rpy=0 0 0
- added joint fp3_2_finger_joint1: type prismatic, parent fp3_2_hand, child fp3_2_leftfinger, origin xyz=0 0 0.0584 rpy=0 0 0, axis 0 1 0, limit lower=0.0 upper=0.04 effort=100 velocity=0.2
- added joint fp3_2_finger_joint2: type prismatic, parent fp3_2_hand, child fp3_2_rightfinger, origin xyz=0 0 0.0584 rpy=0 0 3.141592653589793, axis 0 1 0, limit lower=0.0 upper=0.04 effort=100 velocity=0.2, mimic joint=fp3_2_finger_joint1
- added joint fp3_2_hand_joint: type fixed, parent fp3_2_link8, child fp3_2_hand, origin xyz=0 0 0 rpy=0 0 -0.7853981633974483
- added joint fp3_2_hand_tcp_joint: type fixed, parent fp3_2_hand, child fp3_2_hand_tcp, origin xyz=0 0 0.1034 rpy=0 0 0
- added joint fp3_2_joint1: type revolute, parent fp3_2_link0, child fp3_2_link1, origin xyz=0 0 0.333 rpy=0 0 0, axis 0 0 1, limit lower=-2.7437 upper=2.7437 effort=87.0 velocity=2.62
- added joint fp3_2_joint2: type revolute, parent fp3_2_link1, child fp3_2_link2, origin xyz=0 0 0 rpy=-1.570796326794897 0 0, axis 0 0 1, limit lower=-1.7837 upper=1.7837 effort=87.0 velocity=2.62
- added joint fp3_2_joint3: type revolute, parent fp3_2_link2, child fp3_2_link3, origin xyz=0 -0.316 0 rpy=1.570796326794897 0 0, axis 0 0 1, limit lower=-2.9007 upper=2.9007 effort=87.0 velocity=2.62
- added joint fp3_2_joint4: type revolute, parent fp3_2_link3, child fp3_2_link4, origin xyz=0.0825 0 0 rpy=1.570796326794897 0 0, axis 0 0 1, limit lower=-3.0421 upper=-0.1518 effort=87.0 velocity=2.62
- added joint fp3_2_joint5: type revolute, parent fp3_2_link4, child fp3_2_link5, origin xyz=-0.0825 0.384 0 rpy=-1.570796326794897 0 0, axis 0 0 1, limit lower=-2.8065 upper=2.8065 effort=12.0 velocity=5.26
- added joint fp3_2_joint6: type revolute, parent fp3_2_link5, child fp3_2_link6, origin xyz=0 0 0 rpy=1.570796326794897 0 0, axis 0 0 1, limit lower=0.5445 upper=4.5169 effort=12.0 velocity=4.18
- added joint fp3_2_joint7: type revolute, parent fp3_2_link6, child fp3_2_link7, origin xyz=0.088 0 0 rpy=1.570796326794897 0 0, axis 0 0 1, limit lower=-3.0159 upper=3.0159 effort=12.0 velocity=5.26
- added joint fp3_2_joint8: type fixed, parent fp3_2_link7, child fp3_2_link8, origin xyz=0 0 0.107 rpy=0 0 0
