Commit message: Fixed urdfs

File: urdf/ur5.urdf (robot description, URDF)
Before this commit: robot ur5, 13 links, 12 joints
Links:
- removed link base_link
- removed link base_link_inertia
- removed link forearm_link
- removed link shoulder_link
- removed link upper_arm_link
- removed link wrist_1_link
- removed link wrist_2_link
- removed link wrist_3_link
- added link ur5_link0
- added link ur5_link0_inertia, mass 4.0; collision mesh filename=package://robot_descriptions/meshes/ur5/collision/base.stl; visual mesh filename=package://robot_descriptions/meshes/ur5/visual/base.dae
- added link ur5_link1, mass 3.7; collision mesh filename=package://robot_descriptions/meshes/ur5/collision/shoulder.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; visual mesh filename=package://robot_descriptions/meshes/ur5/visual/shoulder.dae
- added link ur5_link2, mass 8.393; collision mesh filename=package://robot_descriptions/meshes/ur5/collision/upperarm.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; visual mesh filename=package://robot_descriptions/meshes/ur5/visual/upperarm.dae
- added link ur5_link3, mass 2.33; collision mesh filename=package://robot_descriptions/meshes/ur5/collision/forearm.s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; visual mesh filename=package://robot_descriptions/meshes/ur5/visual/forearm.dae
- added link ur5_link4, mass 1.219; collision mesh filename=package://robot_descriptions/meshes/ur5/collision/wrist1.stl; visual mesh filename=package://robot_descriptions/meshes/ur5/visual/wrist1.dae
- added link ur5_link5, mass 1.219; collision mesh filename=package://robot_descriptions/meshes/ur5/collision/wrist2.stl; visual mesh filename=package://robot_descriptions/meshes/ur5/visual/wrist2.dae
- added link ur5_link6, mass 0.1879; collision mesh filename=package://robot_descriptions/meshes/ur5/collision/wrist3.stl; visual mesh filename=package://robot_descriptions/meshes/ur5/visual/wrist3.dae
Joints:
- removed joint base_joint
- removed joint base_link-base_fixed_joint
- removed joint base_link-base_link_inertia
- removed joint elbow_joint
- removed joint shoulder_lift_joint
- removed joint shoulder_pan_joint
- removed joint wrist_1_joint
- removed joint wrist_2_joint
- removed joint wrist_3_joint
- removed joint wrist_3_link-ft_frame
- added joint ur5_base_joint: type fixed, parent world, child ur5_link0, origin xyz=0 0 0 rpy=0 0 0
- added joint ur5_base_link-ur5_base_link_inertia: type fixed, parent ur5_link0, child ur5_link0_inertia, origin xyz=0 0 0 rpy=0 0 3.141592653589793
- added joint ur5_joint1: type revolute, parent ur5_link0_inertia, child ur5_link1, origin xyz=0 0 0.089159 rpy=0 0 0, axis 0 0 1, limit lower=-6.283185307179586 upper=6.283185307179586 effort=150.0 velocity=3.141592653589793
- added joint ur5_joint2: type revolute, parent ur5_link1, child ur5_link2, origin xyz=0 0 0 rpy=1.570796327 0 0, axis 0 0 1, limit lower=-6.283185307179586 upper=6.283185307179586 effort=150.0 velocity=3.141592653589793
- added joint ur5_joint3: type revolute, parent ur5_link2, child ur5_link3, origin xyz=-0.425 0 0 rpy=0 0 0, axis 0 0 1, limit lower=-3.141592653589793 upper=3.141592653589793 effort=150.0 velocity=3.141592653589793
- added joint ur5_joint4: type revolute, parent ur5_link3, child ur5_link4, origin xyz=-0.39225 0 0.10915 rpy=0 0 0, axis 0 0 1, limit lower=-6.283185307179586 upper=6.283185307179586 effort=28.0 velocity=3.141592653589793
- added joint ur5_joint5: type revolute, parent ur5_link4, child ur5_link5, origin xyz=0 -0.09465 -1.941303950897609e-11 rpy=1.570796327 0 0, axis 0 0 1, limit lower=-6.283185307179586 upper=6.283185307179586 effort=28.0 velocity=3.141592653589793
- added joint ur5_joint6: type revolute, parent ur5_link5, child ur5_link6, origin xyz=0 0.0823 -1.688001216681175e-11 rpy=1.570796326589793 3.141592653589793 3.141592653589793, axis 0 0 1, limit lower=-6.283185307179586 upper=6.283185307179586 effort=28.0 velocity=3.141592653589793
- added joint ur5_link0-ur5_base_fixed_joint: type fixed, parent ur5_link0, child base, origin xyz=0 0 0 rpy=0 0 3.141592653589793
- added joint ur5_link6-ft_frame: type fixed, parent ur5_link6, child ft_frame, origin xyz=0 0 0 rpy=3.141592653589793 0 0
- joint wrist_3-flange: parent wrist_3_link -> ur5_link6
